File: doc/PixiePico.kicad_sch (KiCad schematic)
At the start: 20 parts, among them J1 SPKR, J2 MIC, J3 Antenna, J4 Jack-DC, Q1 2N7000, Q2 2N7000, U1 rp2040-zero, U2 Si5351A-B-GT, U3 L7805

Commit message: design
Parts:
- removed PCB: ~, symbol mcu:PixieZ
- added C10, C9: 100uF/16V, symbol Device:C_Polarized
- added C2, C5: 100n, symbol Device:C
- added C6: 10u/16V, symbol Device:C_Polarized
- added C7, C8: 10nF, symbol Device:C
- added L1: 100uH, symbol Device:L
- added U4: ~, symbol mcu:PixieZ
- Q1, Q2: value 2N7000 -> BS170
- R2: value 10K -> 20K
- R3: value 1M -> 20K
Connections:
- net GND: now also C10.2, C2.2, C5.2, C6.2, C7.2, C9.2
- net at R3.1, R7.1, U1.21 (3V3)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: now also C2.1
- net at U2.6 (CLK2): now also U1.12 (11)
- net at Q1.2 (G), R1.1: now also U1.3 (2); no longer U1.6 (5)
- net at Q2.3 (D), R7.2: now also U1.18 (27); no longer U1.17 (26)
- net at U1.23 (5V), U3.3 (OUT): now also C5.1, C6.1
- net at U3.1 (IN): now also C7.1, C9.1, L1.1
- new net: C10.1, C8.1, L1.2
Other:
- note added: "CAL"
- note added: "FSK"
- note added: "PTT"
- note added: "SCL"
- note added: "SDA"
- company: (none) -> LU7DZ
- title: (none) -> PixiePico
- moved on the sheet: C1, C3, C4, Q2, R2, R3, R4, R5, R6, R7, U3

Commit message: design
Parts:
- added M1: Fan, symbol Motor:Fan
- added Q3: BS107, Package_TO_SOT_THT:TO-92_Inline, symbol Transistor_FET:BS107
- added R8: 100K, symbol Device:R
Connections:
- net GND: now also M1.2 (-), R8.2
- net at C5.1, C6.1, U1.23 (5V)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: now also Q3.1 (D)
- net at U1.6 (5): now also Q3.2 (G), R8.1
- new net: M1.1 (+), Q3.3 (S)
Other:
- note added: "FAN"
Changed lines of the file:
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@@
   (junction (at 100.33 76.2) (diameter 0) (color 0 0 0 0)
   )
+  (junction (at 44.45 91.44) (diameter 0) (color 0 0 0 0)
+  )
   (junction (at 66.04 147.32) (diameter 0) (color 0 0 0 0)
   )
@@
   (junction (at 73.66 152.4) (diameter 0) (color 0 0 0 0)
   )
+  (junction (at 58.42 68.58) (diameter 0) (color 0 0 0 0)
+  )
   (junction (at 113.03 118.11) (diameter 0) (color 0 0 0 0)
   )
@@
     (stroke (width 0) (type default))
   )
+  (wire (pts (xy 109.22 102.87) (xy 50.8 102.87))
+    (stroke (width 0) (type default))
+  )
+  (wire (pts (xy 40.64 91.44) (xy 44.45 91.44))
+    (stroke (width 0) (type default))
+  )
   (wire (pts (xy 104.14 152.4) (xy 99.06 152.4))
     (stroke (width 0) (type default))
@@
     (stroke (width 0) (type default))
   )
+  (wire (pts (xy 50.8 102.87) (xy 50.8 91.44))
+    (stroke (width 0) (type default))
+  )
   (wire (pts (xy 224.79 91.44) (xy 231.14 91.44))
     (stroke (width 0) (type default))
   )
+  (wire (pts (xy 100.33 81.28) (xy 109.22 81.28))
+    (stroke (width 0) (type default))
+  )
   (wire (pts (xy 116.84 147.32) (xy 116.84 152.4))
     (stroke (width 0) (type default))
@@
     (stroke (width 0) (type default))
   )
+  (wire (pts (xy 33.02 68.58) (xy 58.42 68.58))
+    (stroke (width 0) (type default))
+  )
   (wire (pts (xy 119.38 52.07) (xy 148.59 52.07))
     (stroke (width 0) (type default))
@@
     (stroke (width 0) (type default))
   )
+  (wire (pts (xy 44.45 91.44) (xy 50.8 91.44))
+    (stroke (width 0) (type default))
+  )
   (wire (pts (xy 111.76 86.36) (xy 127 86.36))
     (stroke (width 0) (type default))
@@
     (stroke (width 0) (type default))
   )
+  (wire (pts (xy 109.22 81.28) (xy 109.22 102.87))
+    (stroke (width 0) (type default))
+  )
   (wire (pts (xy 226.06 67.31) (xy 242.57 67.31))
     (stroke (width 0) (type default))
@@
     (stroke (width 0) (type default))
   )
+  (wire (pts (xy 33.02 86.36) (xy 33.02 68.58))
+    (stroke (width 0) (type default))
+  )
   (wire (pts (xy 100.33 73.66) (xy 119.38 73.66))
     (stroke (width 0) (type default))
@@
   (wire (pts (xy 231.14 91.44) (xy 231.14 93.98))
     (stroke (width 0) (type default))
+  )
+  (text "FAN" (at 101.6 81.28 0)
+    (effects (font (size 1.27 1.27)) (justify left bottom))
   )
   (text "PTT" (at 101.6 73.66 0)
@@
     )
   )
+  (symbol (lib_id "Motor:Fan") (at 33.02 104.14 0) (unit 1)
+    (in_bom yes) (on_board yes) (dnp no) (fields_autoplaced)
+    (property "Reference" "M1" (at 38.1 103.505 0)
+      (effects (font (size 1.27 1.27)) (justify left))
+    )
+    (property "Value" "Fan" (at 38.1 106.045 0)
+      (effects (font (size 1.27 1.27)) (justify left))
+    )
+    (property "Footprint" "" (at 33.02 103.886 0)
+      (effects (font (size 1.27 1.27)) hide)
+    )
+    (property "Datasheet" "~" (at 33.02 103.886 0)
+      (effects (font (size 1.27 1.27)) hide)
+    )
+    (pin "1")
+    (pin "2")
+    (instances
+      (project "PixiePico"
+        (path "/a432cb18-7a14-49a3-8d10-48c0fec11b89"
+          (reference "M1") (unit 1)
+        )
+      )
+    )
+  )
+  (symbol (lib_name "GND_2") (lib_id "power:GND") (at 33.02 109.22 0) (unit 1)
+    (in_bom yes) (on_board yes) (dnp no)
+    (property "Reference" "#PWR021" (at 33.02 115.57 0)
+      (effects (font (size 1.27 1.27)) hide)
+    )
+    (property "Value" "GND" (at 33.02 137.16 0)
+      (effects (font (size 1.27 1.27)) hide)
+    )
+    (property "Footprint" "" (at 33.02 109.22 0)
+      (effects (font (size 1.27 1.27)) hide)
+    )
+    (property "Datasheet" "" (at 33.02 109.22 0)
+      (effects (font (size 1.27 1.27)) hide)
+    )
+    (pin "1")
+    (instances
+      (project "PixiePico"
+        (path "/a432cb18-7a14-49a3-8d10-48c0fec11b89"
+          (reference "#PWR021") (unit 1)
+        )
+      )
+    )
+  )
   (symbol (lib_name "GND_18") (lib_id "power:GND") (at 218.44 53.34 0) (unit 1)
     (in_bom yes) (on_board yes) (dnp no) (fields_autoplaced)
@@
         (path "/a432cb18-7a14-49a3-8d10-48c0fec11b89"
           (reference "#PWR05") (unit 1)
+        )
+      )
+    )
+  )
+  (symbol (lib_id "Device:R") (at 44.45 95.25 0) (unit 1)
+    (in_bom yes) (on_board yes) (dnp no) (fields_autoplaced)
+    (property "Reference" "R8" (at 46.99 94.615 0)
+      (effects (font (size 1.27 1.27)) (justify left))
+    )
+    (property "Value" "100K" (at 46.99 97.155 0)
+      (effects (font (size 1.27 1.27)) (justify left))
+    )
+    (property "Footprint" "" (at 42.672 95.25 90)
+      (effects (font (size 1.27 1.27)) hide)
+    )
+    (property "Datasheet" "~" (at 44.45 95.25 0)
+      (effects (font (size 1.27 1.27)) hide)
+    )
+    (pin "1")
+    (pin "2")
+    (instances
+      (project "PixiePico"
+        (path "/a432cb18-7a14-49a3-8d10-48c0fec11b89"
+          (reference "R8") (unit 1)
         )
       )
@@
         (path "/a432cb18-7a14-49a3-8d10-48c0fec11b89"
           (reference "J1") (unit 1)
+        )
+      )
+    )
+  )
+  (symbol (lib_name "GND_2") (lib_id "power:GND") (at 44.45 99.06 0) (unit 1)
+    (in_bom yes) (on_board yes) (dnp no)
+    (property "Reference" "#PWR020" (at 44.45 105.41 0)
+      (effects (font (size 1.27 1.27)) hide)
+    )
+    (property "Value" "GND" (at 44.45 127 0)
+      (effects (font (size 1.27 1.27)) hide)
+    )
+    (property "Footprint" "" (at 44.45 99.06 0)
+      (effects (font (size 1.27 1.27)) hide)
+    )
+    (property "Datasheet" "" (at 44.45 99.06 0)
+      (effects (font (size 1.27 1.27)) hide)
+    )
+    (pin "1")
+    (instances
+      (project "PixiePico"
+        (path "/a432cb18-7a14-49a3-8d10-48c0fec11b89"
+          (reference "#PWR020") (unit 1)
         )
       )
@@
         )
       )
+    )
+  )
+  (symbol (lib_id "Transistor_FET:BS107") (at 35.56 91.44 0) (mirror y) (unit 1)
+    (in_bom yes) (on_board yes) (dnp no)
+    (property "Reference" "Q3" (at 29.21 90.805 0)
+      (effects (font (size 1.27 1.27)) (justify left))
+    )
+    (property "Value" "BS107" (at 29.21 93.345 0)
+      (effects (font (size 1.27 1.27)) (justify left))
+    )
+    (property "Footprint" "Package_TO_SOT_THT:TO-92_Inline" (at 30.48 93.345 0)
+      (effects (font (size 1.27 1.27) italic) (justify left) hide)
+    )
+    (property "Datasheet" "http://www.onsemi.com/pub_link/Collateral/BS107-D.PDF" (at 35.56 91.44 0)
+      (effects (font (size 1.27 1.27)) (justify left) hide)
+    )
+    (pin "1")
+    (pin "2")
+    (pin "3")
+    (instances
+      (project "PixiePico"
+        (path "/a432cb18-7a14-49a3-8d10-48c0fec11b89"
+          (reference "Q3") (unit 1)
+        )
+      )

Commit message: design
Parts:
- removed C3, C4: 10n, symbol Device:C
- removed Q2: BS170, Package_TO_SOT_THT:TO-92_Inline, symbol Transistor_FET:2N7000
- removed R4, R5: 10K, symbol Device:R
- removed R6: 100K, symbol Device:R
- removed R7: 1K, symbol Device:R
- C1: value 100n -> 4.7u
- R2, R3: value 20K -> 10K
Connections:
- net GND: now also R3.2; no longer R2.1
- net at C2.1, U1.21 (3V3), U2.1 (VDD): now also R2.1; no longer R3.1
- net at U1.17 (26): now also C1.1, R2.2, R3.1
- now unconnected: C1.2
Other:
- note removed: "FSK"

Commit message: PixiePico
Other:
- note added: "+5V"
- note added: "AUDIO"
Changed lines of the file:
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@@
     (stroke (width 0) (type default))
+  )
+  (text "AUDIO" (at 67.31 83.82 0)
+    (effects (font (size 1.27 1.27)) (justify left bottom))
   )
   (text "FAN" (at 101.6 81.28 0)
@@
     (effects (font (size 1.27 1.27)) (justify left bottom))
   )
+  (text "+5V" (at 68.58 68.58 0)
+    (effects (font (size 1.27 1.27)) (justify left bottom))
+  )

Commit message: Design
Parts:
- added R4: 10K, symbol Device:R
- added SW1: TXSW, symbol Switch:SW_Push
Connections:
- net GND: now also SW1.1
- net at C1.1, R2.2, R3.1: now also U1.18 (27); no longer U1.17 (26)
- net at C2.1, R2.1, U1.21 (3V3)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: now also R4.2
- net at U1.9 (8): now also R4.1, SW1.2
Other:
- note added: "FSKin"
- note added: "RXSW"
- note added: "TXSW"
- note removed: "AUDIO"
- note removed: "PTT"
Changed lines of the file:
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@@
   (junction (at 66.04 73.66) (diameter 0) (color 0 0 0 0)
   )
-  (junction (at 66.04 83.82) (diameter 0) (color 0 0 0 0)
-  )
   (junction (at 109.22 59.69) (diameter 0) (color 0 0 0 0)
   )
+  (junction (at 74.93 81.28) (diameter 0) (color 0 0 0 0)
+  )
+  (junction (at 100.33 76.2) (diameter 0) (color 0 0 0 0)
+  )
   (junction (at 142.24 118.11) (diameter 0) (color 0 0 0 0)
   )
+  (junction (at 44.45 91.44) (diameter 0) (color 0 0 0 0)
+  )
+  (junction (at 74.93 118.11) (diameter 0) (color 0 0 0 0)
+  )
+  (junction (at 66.04 81.28) (diameter 0) (color 0 0 0 0)
+  )
+  (junction (at 231.14 78.74) (diameter 0) (color 0 0 0 0)
+  )
   (junction (at 100.33 78.74) (diameter 0) (color 0 0 0 0)
   )
-  (junction (at 100.33 76.2) (diameter 0) (color 0 0 0 0)
-  )
-  (junction (at 44.45 91.44) (diameter 0) (color 0 0 0 0)
-  )
-  (junction (at 74.93 118.11) (diameter 0) (color 0 0 0 0)
-  )
-  (junction (at 231.14 78.74) (diameter 0) (color 0 0 0 0)
-  )
   (junction (at 231.14 91.44) (diameter 0) (color 0 0 0 0)
   )
@@
   (junction (at 148.59 52.07) (diameter 0) (color 0 0 0 0)
   )
+  (junction (at 121.92 88.9) (diameter 0) (color 0 0 0 0)
+  )
+  (junction (at 121.92 59.69) (diameter 0) (color 0 0 0 0)
+  )
   (junction (at 87.63 93.98) (diameter 0) (color 0 0 0 0)
   )
@@
     (stroke (width 0) (type default))
   )
+  (wire (pts (xy 121.92 59.69) (xy 121.92 64.77))
+    (stroke (width 0) (type default))
+  )
   (wire (pts (xy 74.93 73.66) (xy 66.04 73.66))
     (stroke (width 0) (type default))
@@
     (stroke (width 0) (type default))
   )
-  (wire (pts (xy 76.2 81.28) (xy 74.93 81.28))
+  (wire (pts (xy 66.04 81.28) (xy 74.93 81.28))
     (stroke (width 0) (type default))
   )
@@
     (stroke (width 0) (type default))
   )
-  (wire (pts (xy 114.3 76.2) (xy 114.3 88.9))
+  (wire (pts (xy 127 88.9) (xy 125.73 88.9))
     (stroke (width 0) (type default))
   )
@@
     (stroke (width 0) (type default))
   )
+  (wire (pts (xy 125.73 88.9) (xy 125.73 76.2))
+    (stroke (width 0) (type default))
+  )
   (wire (pts (xy 142.24 118.11) (xy 152.4 118.11))
     (stroke (width 0) (type default))
   )
-  (wire (pts (xy 100.33 78.74) (xy 111.76 78.74))
+  (wire (pts (xy 74.93 81.28) (xy 76.2 81.28))
     (stroke (width 0) (type default))
   )
@@
     (stroke (width 0) (type default))
   )
+  (wire (pts (xy 121.92 59.69) (xy 137.16 59.69))
+    (stroke (width 0) (type default))
+  )
   (wire (pts (xy 99.06 73.66) (xy 100.33 73.66))
     (stroke (width 0) (type default))
   )
-  (wire (pts (xy 62.23 83.82) (xy 62.23 109.22))
+  (wire (pts (xy 62.23 81.28) (xy 62.23 109.22))
     (stroke (width 0) (type default))
   )
@@
     (stroke (width 0) (type default))
   )
-  (wire (pts (xy 66.04 83.82) (xy 74.93 83.82))
-    (stroke (width 0) (type default))
-  )
   (wire (pts (xy 66.04 59.69) (xy 109.22 59.69))
     (stroke (width 0) (type default))
@@
     (stroke (width 0) (type default))
   )
+  (wire (pts (xy 100.33 78.74) (xy 123.19 78.74))
+    (stroke (width 0) (type default))
+  )
   (wire (pts (xy 204.47 48.26) (xy 204.47 62.23))
     (stroke (width 0) (type default))
@@
     (stroke (width 0) (type default))
   )
+  (wire (pts (xy 123.19 86.36) (xy 123.19 78.74))
+    (stroke (width 0) (type default))
+  )
   (wire (pts (xy 148.59 59.69) (xy 148.59 64.77))
     (stroke (width 0) (type default))
   )
-  (wire (pts (xy 66.04 81.28) (xy 66.04 83.82))
+  (wire (pts (xy 66.04 81.28) (xy 66.04 85.09))
     (stroke (width 0) (type default))
   )
@@
     (stroke (width 0) (type default))
   )
+  (wire (pts (xy 175.26 59.69) (xy 175.26 67.31))
+    (stroke (width 0) (type default))
+  )
+  (wire (pts (xy 137.16 59.69) (xy 137.16 68.58))
+    (stroke (width 0) (type default))
+  )
+  (wire (pts (xy 231.14 78.74) (xy 231.14 81.28))
+    (stroke (width 0) (type default))
+  )
   (wire (pts (xy 100.33 81.28) (xy 109.22 81.28))
     (stroke (width 0) (type default))
   )
-  (wire (pts (xy 175.26 59.69) (xy 175.26 67.31))
-    (stroke (width 0) (type default))
-  )
-  (wire (pts (xy 137.16 59.69) (xy 137.16 68.58))
-    (stroke (width 0) (type default))
-  )
-  (wire (pts (xy 231.14 78.74) (xy 231.14 81.28))
-    (stroke (width 0) (type default))
-  )
   (wire (pts (xy 158.75 105.41) (xy 87.63 105.41))
     (stroke (width 0) (type default))
@@
     (stroke (width 0) (type default))
   )
+  (wire (pts (xy 62.23 81.28) (xy 66.04 81.28))
+    (stroke (width 0) (type default))
+  )
   (wire (pts (xy 58.42 68.58) (xy 74.93 68.58))
     (stroke (width 0) (type default))
@@
     (stroke (width 0) (type default))
   )
-  (wire (pts (xy 111.76 78.74) (xy 111.76 86.36))
-    (stroke (width 0) (type default))
-  )
   (wire (pts (xy 151.13 76.2) (xy 152.4 76.2))
     (stroke (width 0) (type default))
@@
     (stroke (width 0) (type default))
   )
+  (wire (pts (xy 127 86.36) (xy 123.19 86.36))
+    (stroke (width 0) (type default))
+  )
   (wire (pts (xy 139.7 118.11) (xy 142.24 118.11))
     (stroke (width 0) (type default))
   )
-  (wire (pts (xy 66.04 83.82) (xy 66.04 85.09))
-    (stroke (width 0) (type default))
-  )
-  (wire (pts (xy 100.33 76.2) (xy 114.3 76.2))
+  (wire (pts (xy 100.33 88.9) (xy 121.92 88.9))
     (stroke (width 0) (type default))
   )
@@
     (stroke (width 0) (type default))
   )
-  (wire (pts (xy 111.76 86.36) (xy 127 86.36))
-    (stroke (width 0) (type default))
-  )
   (wire (pts (xy 105.41 125.73) (xy 105.41 127))
     (stroke (width 0) (type default))
   )
+  (wire (pts (xy 121.92 72.39) (xy 121.92 88.9))
+    (stroke (width 0) (type default))
+  )
   (wire (pts (xy 66.04 73.66) (xy 66.04 59.69))
     (stroke (width 0) (type default))
@@
     (stroke (width 0) (type default))
   )
+  (wire (pts (xy 100.33 76.2) (xy 125.73 76.2))
+    (stroke (width 0) (type default))
+  )
   (wire (pts (xy 97.79 118.11) (xy 86.36 118.11))
     (stroke (width 0) (type default))
@@
     (stroke (width 0) (type default))
   )
-  (wire (pts (xy 114.3 88.9) (xy 127 88.9))
-    (stroke (width 0) (type default))
-  )
-  (wire (pts (xy 66.04 83.82) (xy 62.23 83.82))
-    (stroke (width 0) (type default))
-  )
   (wire (pts (xy 109.22 81.28) (xy 109.22 102.87))
     (stroke (width 0) (type default))
@@
     (stroke (width 0) (type default))
   )
-  (wire (pts (xy 109.22 59.69) (xy 137.16 59.69))
+  (wire (pts (xy 109.22 59.69) (xy 121.92 59.69))
     (stroke (width 0) (type default))
   )
@@
     (stroke (width 0) (type default))
   )
-  (text "AUDIO" (at 67.31 83.82 0)
+  (text "FSKin" (at 67.31 83.82 0)
     (effects (font (size 1.27 1.27)) (justify left bottom))
   )
@@
     (effects (font (size 1.27 1.27)) (justify left bottom))
   )
-  (text "PTT" (at 101.6 73.66 0)
+  (text "RXSW" (at 101.6 73.66 0)
     (effects (font (size 1.27 1.27)) (justify left bottom))
   )
@@
   )
   (text "+5V" (at 68.58 68.58 0)
+    (effects (font (size 1.27 1.27)) (justify left bottom))
+  )
+  (text "TXSW" (at 101.6 88.9 0)
     (effects (font (size 1.27 1.27)) (justify left bottom))
   )
@@
     )
   )
+  (symbol (lib_id "Device:R") (at 121.92 68.58 180) (unit 1)
+    (in_bom yes) (on_board yes) (dnp no) (fields_autoplaced)
+    (property "Reference" "R4" (at 124.46 67.945 0)
+      (effects (font (size 1.27 1.27)) (justify right))
+    )
+    (property "Value" "10K" (at 124.46 70.485 0)
+      (effects (font (size 1.27 1.27)) (justify right))
+    )
+    (property "Footprint" "" (at 123.698 68.58 90)
+      (effects (font (size 1.27 1.27)) hide)
+    )
+    (property "Datasheet" "~" (at 121.92 68.58 0)
+      (effects (font (size 1.27 1.27)) hide)
+    )
+    (pin "1")
+    (pin "2")
+    (instances
+      (project "PixiePico"
+        (path "/a432cb18-7a14-49a3-8d10-48c0fec11b89"
+          (reference "R4") (unit 1)
+        )
+      )
+    )
+  )
   (symbol (lib_id "Transistor_FET:2N7000") (at 161.29 57.15 270) (unit 1)
     (in_bom yes) (on_board yes) (dnp no)
@@
     )
   )
+  (symbol (lib_id "Switch:SW_Push") (at 121.92 93.98 90) (unit 1)
+    (in_bom yes) (on_board yes) (dnp no) (fields_autoplaced)
+    (property "Reference" "SW1" (at 123.19 93.345 90)
+      (effects (font (size 1.27 1.27)) (justify right))
+    )
+    (property "Value" "TXSW" (at 123.19 95.885 90)
+      (effects (font (size 1.27 1.27)) (justify right))
+    )
+    (property "Footprint" "" (at 116.84 93.98 0)
+      (effects (font (size 1.27 1.27)) hide)
+    )
+    (property "Datasheet" "~" (at 116.84 93.98 0)
+      (effects (font (size 1.27 1.27)) hide)
+    )
+    (pin "1")
+    (pin "2")
+    (instances
+      (project "PixiePico"
+        (path "/a432cb18-7a14-49a3-8d10-48c0fec11b89"
+          (reference "SW1") (unit 1)
+        )
+      )
+    )
+  )
   (symbol (lib_id "Connector_Audio:AudioJack2") (at 236.22 93.98 0) (mirror y) (unit 1)
     (in_bom yes) (on_board yes) (dnp no)
@@
         )
       )
+    )
+  )
+  (symbol (lib_name "GND_11") (lib_id "power:GND") (at 121.92 99.06 0) (unit 1)
+    (in_bom yes) (on_board yes) (dnp no) (fields_autoplaced)
+    (property "Reference" "#PWR09" (at 121.92 105.41 0)
+      (effects (font (size 1.27 1.27)) hide)
+    )
+    (property "Value" "GND" (at 121.92 104.14 0)
+      (effects (font (size 1.27 1.27)) hide)
+    )
+    (property "Footprint" "" (at 121.92 99.06 0)
+      (effects (font (size 1.27 1.27)) hide)
+    )
+    (property "Datasheet" "" (at 121.92 99.06 0)
+      (effects (font (size 1.27 1.27)) hide)
+    )
+    (pin "1")
+    (instances
+      (project "PixiePico"
+        (path "/a432cb18-7a14-49a3-8d10-48c0fec11b89"
+          (reference "#PWR09") (unit 1)
+        )
+      )
