File: doc/PixiePico.kicad_sch (KiCad schematic)
At the start: 26 parts, among them J1 SPKR, J2 MIC, J3 Antenna, J4 Jack-DC, M1 Fan, Q1 BS170, Q3 BS107, SW1 TXSW, U1 rp2040-zero, U2 Si5351A-B-GT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

Commit message: Design
Parts:
- removed U2: Si5351A-B-GT, Package_SO:MSOP-10_3x3mm_P0.5mm, symbol Oscillator:Si5351A-B-GT
- added C3: 10nF, symbol Device:C
Connections:
- net at U1.7 (6): now also C3.1
Changed lines of the file:
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@@
   (junction (at 148.59 59.69) (diameter 0) (color 0 0 0 0)
   )
-  (junction (at 152.4 76.2) (diameter 0) (color 0 0 0 0)
-  )
   (junction (at 127 119.38) (diameter 0) (color 0 0 0 0)
   )
@@
   (junction (at 74.93 81.28) (diameter 0) (color 0 0 0 0)
   )
-  (junction (at 100.33 76.2) (diameter 0) (color 0 0 0 0)
-  )
   (junction (at 142.24 118.11) (diameter 0) (color 0 0 0 0)
   )
@@
   (junction (at 231.14 78.74) (diameter 0) (color 0 0 0 0)
   )
-  (junction (at 100.33 78.74) (diameter 0) (color 0 0 0 0)
-  )
   (junction (at 231.14 91.44) (diameter 0) (color 0 0 0 0)
   )
@@
   (junction (at 121.92 88.9) (diameter 0) (color 0 0 0 0)
   )
-  (junction (at 121.92 59.69) (diameter 0) (color 0 0 0 0)
-  )
-  (junction (at 87.63 93.98) (diameter 0) (color 0 0 0 0)
-  )
   (junction (at 86.36 118.11) (diameter 0) (color 0 0 0 0)
   )
@@
     (stroke (width 0) (type default))
   )
+  (wire (pts (xy 133.35 76.2) (xy 146.05 76.2))
+    (stroke (width 0) (type default))
+  )
   (wire (pts (xy 66.04 81.28) (xy 74.93 81.28))
     (stroke (width 0) (type default))
   )
-  (wire (pts (xy 152.4 86.36) (xy 158.75 86.36))
-    (stroke (width 0) (type default))
-  )
-  (wire (pts (xy 127 88.9) (xy 125.73 88.9))
+  (wire (pts (xy 100.33 83.82) (xy 133.35 83.82))
     (stroke (width 0) (type default))
   )
@@
     (stroke (width 0) (type default))
   )
-  (wire (pts (xy 125.73 88.9) (xy 125.73 76.2))
-    (stroke (width 0) (type default))
-  )
   (wire (pts (xy 142.24 118.11) (xy 152.4 118.11))
     (stroke (width 0) (type default))
@@
     (stroke (width 0) (type default))
   )
+  (wire (pts (xy 153.67 76.2) (xy 184.15 76.2))
+    (stroke (width 0) (type default))
+  )
   (wire (pts (xy 204.47 99.06) (xy 204.47 101.6))
     (stroke (width 0) (type default))
@@
     (stroke (width 0) (type default))
   )
-  (wire (pts (xy 121.92 59.69) (xy 137.16 59.69))
-    (stroke (width 0) (type default))
-  )
   (wire (pts (xy 99.06 73.66) (xy 100.33 73.66))
     (stroke (width 0) (type default))
@@
     (stroke (width 0) (type default))
   )
-  (wire (pts (xy 87.63 93.98) (xy 87.63 105.41))
-    (stroke (width 0) (type default))
-  )
   (wire (pts (xy 173.99 91.44) (xy 185.42 91.44))
     (stroke (width 0) (type default))
@@
     (stroke (width 0) (type default))
   )
-  (wire (pts (xy 100.33 78.74) (xy 123.19 78.74))
-    (stroke (width 0) (type default))
-  )
   (wire (pts (xy 204.47 48.26) (xy 204.47 62.23))
     (stroke (width 0) (type default))
@@
     (stroke (width 0) (type default))
   )
-  (wire (pts (xy 139.7 93.98) (xy 139.7 96.52))
-    (stroke (width 0) (type default))
-  )
-  (wire (pts (xy 123.19 86.36) (xy 123.19 78.74))
-    (stroke (width 0) (type default))
-  )
   (wire (pts (xy 148.59 59.69) (xy 148.59 64.77))
     (stroke (width 0) (type default))
@@
     (stroke (width 0) (type default))
   )
-  (wire (pts (xy 152.4 76.2) (xy 184.15 76.2))
-    (stroke (width 0) (type default))
-  )
   (wire (pts (xy 50.8 102.87) (xy 50.8 91.44))
     (stroke (width 0) (type default))
@@
     (stroke (width 0) (type default))
   )
-  (wire (pts (xy 137.16 59.69) (xy 137.16 68.58))
-    (stroke (width 0) (type default))
-  )
   (wire (pts (xy 231.14 78.74) (xy 231.14 81.28))
     (stroke (width 0) (type default))
@@
     (stroke (width 0) (type default))
   )
-  (wire (pts (xy 158.75 105.41) (xy 87.63 105.41))
-    (stroke (width 0) (type default))
-  )
   (wire (pts (xy 173.99 91.44) (xy 173.99 109.22))
     (stroke (width 0) (type default))
@@
     (stroke (width 0) (type default))
   )
-  (wire (pts (xy 151.13 76.2) (xy 152.4 76.2))
-    (stroke (width 0) (type default))
-  )
   (wire (pts (xy 152.4 118.11) (xy 152.4 119.38))
     (stroke (width 0) (type default))
   )
-  (wire (pts (xy 127 86.36) (xy 123.19 86.36))
-    (stroke (width 0) (type default))
-  )
   (wire (pts (xy 139.7 118.11) (xy 142.24 118.11))
     (stroke (width 0) (type default))
@@
     (stroke (width 0) (type default))
   )
-  (wire (pts (xy 100.33 76.2) (xy 125.73 76.2))
-    (stroke (width 0) (type default))
-  )
   (wire (pts (xy 97.79 118.11) (xy 86.36 118.11))
     (stroke (width 0) (type default))
@@
     (stroke (width 0) (type default))
   )
+  (wire (pts (xy 133.35 83.82) (xy 133.35 76.2))
+    (stroke (width 0) (type default))
+  )
   (wire (pts (xy 218.44 53.34) (xy 227.33 53.34))
-    (stroke (width 0) (type default))
-  )
-  (wire (pts (xy 158.75 86.36) (xy 158.75 105.41))
     (stroke (width 0) (type default))
   )
@@
     )
   )
-  (symbol (lib_id "Oscillator:Si5351A-B-GT") (at 139.7 81.28 0) (unit 1)
-    (in_bom yes) (on_board yes) (dnp no) (fields_autoplaced)
-    (property "Reference" "U2" (at 141.6559 93.98 0)
-      (effects (font (size 1.27 1.27)) (justify left))
-    )
-    (property "Value" "Si5351A-B-GT" (at 141.6559 96.52 0)
-      (effects (font (size 1.27 1.27)) (justify left))
-    )
-    (property "Footprint" "Package_SO:MSOP-10_3x3mm_P0.5mm" (at 139.7 101.6 0)
-      (effects (font (size 1.27 1.27)) hide)
-    )
-    (property "Datasheet" "https://www.silabs.com/documents/public/data-sheets/Si5351-B.pdf" (at 130.81 83.82 0)
-      (effects (font (size 1.27 1.27)) hide)
-    )
-    (pin "1")
-    (pin "10")
-    (pin "2")
-    (pin "3")
-    (pin "4")
-    (pin "5")
-    (pin "6")
-    (pin "7")
-    (pin "8")
-    (pin "9")
-    (instances
-      (project "PixiePico"
-        (path "/a432cb18-7a14-49a3-8d10-48c0fec11b89"
-          (reference "U2") (unit 1)
-        )
-      )
-    )
-  )
   (symbol (lib_id "Device:R") (at 148.59 55.88 0) (unit 1)
     (in_bom yes) (on_board yes) (dnp no) (fields_autoplaced)
@@
     )
     (property "Value" "GND" (at 148.59 69.85 0)
-      (effects (font (size 1.27 1.27)))
+      (effects (font (size 1.27 1.27)) hide)
     )
     (property "Footprint" "" (at 148.59 64.77 0)
@@
     )
   )
-  (symbol (lib_name "GND_15") (lib_id "power:GND") (at 139.7 96.52 0) (unit 1)
-    (in_bom yes) (on_board yes) (dnp no) (fields_autoplaced)
-    (property "Reference" "#PWR01" (at 139.7 102.87 0)
-      (effects (font (size 1.27 1.27)) hide)
-    )
-    (property "Value" "GND" (at 139.7 101.6 0)
-      (effects (font (size 1.27 1.27)) hide)
-    )
-    (property "Footprint" "" (at 139.7 96.52 0)
-      (effects (font (size 1.27 1.27)) hide)
-    )
-    (property "Datasheet" "" (at 139.7 96.52 0)
-      (effects (font (size 1.27 1.27)) hide)
-    )
-    (pin "1")
-    (instances
-      (project "PixiePico"
-        (path "/a432cb18-7a14-49a3-8d10-48c0fec11b89"
-          (reference "#PWR01") (unit 1)
-        )
-      )
+  (symbol (lib_id "Device:C") (at 149.86 76.2 90) (unit 1)
+    (in_bom yes) (on_board yes) (dnp no) (fields_autoplaced)
+    (property "Reference" "C3" (at 149.86 69.85 90)
+      (effects (font (size 1.27 1.27)))
+    )
+    (property "Value" "10nF" (at 149.86 72.39 90)
+      (effects (font (size 1.27 1.27)))
+    )
+    (property "Footprint" "" (at 153.67 75.2348 0)
+      (effects (font (size 1.27 1.27)) hide)
+    )
+    (property "Datasheet" "~" (at 149.86 76.2 0)
+      (effects (font (size 1.27 1.27)) hide)
+    )
+    (pin "1")
+    (pin "2")
+    (instances
+      (project "PixiePico"
+        (path "/a432cb18-7a14-49a3-8d10-48c0fec11b89"
+          (reference "C3") (unit 1)
+        )
+      )

Commit message: dds_rp2040
Parts:
- added R5, R6: 10K, symbol Device:R
- added SW2: UP, symbol Switch:SW_Push
- added SW3: DOWN, symbol Switch:SW_Push
Connections:
- net GND: now also SW2.1, SW3.1
- net FAN: now reaches U1.10 (9)
- net FAN: now also Q3.2 (G), R8.1
- net at C2.1, R2.1, R4.2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: now also R5.2, R6.1
- net at C5.1, C6.1, U1.23 (5V)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: no longer Q3.1 (D)
- net DDS: now reaches C3.1, U1.7 (6)
- net UP: now reaches U1.8 (7)
- net UP: now also R5.1, SW2.2
- new net DOWN: R6.2, SW3.2, U1.6 (5)
Other:
- note removed: "CAL"
- note removed: "FAN"
- moved on the sheet: M1, Q3, R8

Commit message: dds_rp2040
Connections:
- net at C5.1, C6.1, U1.23 (5V)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: now also Q3.1 (D)
Changed lines of the file:
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@@
   (junction (at 152.4 118.11) (diameter 0) (color 0 0 0 0)
   )
-  (junction (at 139.7 59.69) (diameter 0) (color 0 0 0 0)
-  )
   (junction (at 119.38 118.11) (diameter 0) (color 0 0 0 0)
   )
@@
     (stroke (width 0) (type default))
   )
-  (wire (pts (xy 139.7 59.69) (xy 142.24 59.69))
-    (stroke (width 0) (type default))
-  )
   (wire (pts (xy 139.7 72.39) (xy 139.7 81.28))
     (stroke (width 0) (type default))
@@
     (stroke (width 0) (type default))
   )
-  (wire (pts (xy 33.02 86.36) (xy 33.02 68.58))
-    (stroke (width 0) (type default))
-  )
+  (wire (pts (xy 33.02 68.58) (xy 33.02 93.98))
+    (stroke (width 0) (type default))
+  )
