File: doc/PixiePico.kicad_sch (KiCad schematic)
At the start: 30 parts, among them J1 SPKR, J2 MIC, J3 Antenna, J4 Jack-DC, M1 Fan, Q1 BS170, Q3 BS107, SW1 TXSW, SW2 UP, SW3 DOWN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

Commit message: resume project
Parts:
- removed R5, R6: 10K, symbol Device:R
- removed SW2: UP, symbol Switch:SW_Push
- removed SW3: DOWN, symbol Switch:SW_Push
- added SW2: RotaryEncoder, symbol Device:RotaryEncoder
- added U2: SHT1x, Sensor:SHT1x, symbol Sensor:SHT1x
- J2: value MIC -> KEYER
- SW1: value TXSW -> PTT
Connections:
- net DOWN is gone; now on net KEYER: U1.6 (5)
- net DDS: no longer C3.1, U1.7 (6)
- net FAN: now also U1.7 (6); no longer U1.10 (9)
- net GND: now also U2.1 (GND)
- net at C1.2: now also J2.S, J2.T
- net at C2.1, R2.1, R4.2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: now also SW2.C
- net KEYER: now reaches Q1.2 (G), R1.1
- net KEYER: no longer U1.3 (2)
- net at U1.1 (0): now also U1.2 (1), U2.2 (DATA), U2.3 (SCK)
- net at U1.14 (13): now also C3.1
- net at C5.1, C6.1, Q3.1 (D)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: now also U2.4 (VDD)
- net at U1.4 (3): now also SW2.A
- net at U1.5 (4): now also SW2.B
- net at R4.1, SW1.2: now also U1.3 (2); no longer U1.9 (8)
- net at C10.1, C8.1, L1.2: now also J4.2
- net UP: no longer names the net of U1.8 (7)
- no-connect marks 0 -> 1
Other:
- note added: "PTT"
- note added: "ROT1 (Clk)"
- note added: "ROT2 (DT)"
- note removed: "RXSW"
- note removed: "TXSW"
